Commit message: Add audited SNU Bear URDF, mesh assets and simulation guide
Include all ten original CAD meshes as lossless restorable assets, saved poses and crawl samples, explicit X330 assumptions, a PyBullet playback/physics runner and CI smoke checks. Document the distinction between prescribed playback and unvalidated dynamics.

File: motion/src/snu_bear_motion/data/robot/snu_bear_v06.urdf (robot description, URDF)
Before this commit: robot snu_bear_v06_teddy_motion_study, 10 links, 9 joints
Links:
- link head: geometry collision mesh filename=meshes_m/head.stl scale=1 1 1; visual mesh filename=meshes_m/head.stl scale=1 1 1
- link left_fore_lower: geometry collision mesh filename=meshes_m/left_fore_lower.stl scale=1 1 1; visual mesh filename=meshes_m/left_fore_lower.stl scale=1 1 1
- link left_fore_upper: geometry collision mesh filename=meshes_m/left_fore_upper.stl scale=1 1 1; visual mesh filename=meshes_m/left_fore_upper.stl scale=1 1 1
- link left_hind_lower: geometry collision mesh filename=meshes_m/left_hind_lower.stl scale=1 1 1; visual mesh filename=meshes_m/left_hind_lower.stl scale=1 1 1
- link left_hind_upper: geometry collision mesh filename=meshes_m/left_hind_upper.stl scale=1 1 1; visual mesh filename=meshes_m/left_hind_upper.stl scale=1 1 1
- link right_fore_lower: geometry collision mesh filename=meshes_m/right_fore_lower.stl scale=1 1 1; visual mesh filename=meshes_m/right_fore_lower.stl scale=1 1 1
- link right_fore_upper: geometry collision mesh filename=meshes_m/right_fore_upper.stl scale=1 1 1; visual mesh filename=meshes_m/right_fore_upper.stl scale=1 1 1
- link right_hind_lower: geometry collision mesh filename=meshes_m/right_hind_lower.stl scale=1 1 1; visual mesh filename=meshes_m/right_hind_lower.stl scale=1 1 1
- link right_hind_upper: geometry collision mesh filename=meshes_m/right_hind_upper.stl scale=1 1 1; visual mesh filename=meshes_m/right_hind_upper.stl scale=1 1 1
- link torso: geometry collision mesh filename=meshes_m/torso.stl scale=1 1 1; visual mesh filename=meshes_m/torso.stl scale=1 1 1
